Commit message: Delete useless code to collapse dummy links at the root
The code would never execute because a root link would never
be tagged as "dummy" (because it has no supporting joint!).

Also, fixed joints and dummy links at the very start of
the model are already handled by the generic routine for
pruning (collapsing would be better naming).

This code was introduced in 0fd00c0d98c3168d5

I hope I am not missing something here, overlooking
what I thought when I wrote that code.

I also updated the pruning-test with exactly the case
that I thought was special, that is, a fixed joint
between a dummy root and the robot's effective root.
The case is still handled correctly.

File: test/pruning/fixed_joints.urdf (robot description, URDF)
Before this commit: robot dummy_leg, 12 links, 11 joints
Links:
- added link world
Joints:
- added joint world_to_base: type fixed, parent world, child base
